Commit message: added upper arm support

File: urdf/sainsmart_6dof.urdf.xacro (robot description, xacro)
@@ -5,6 +5,9 @@
   <xacro:property name="main_base_dims" value="0.1" />
   <xacro:property name="main_base_height" value="0.01" />
-  <xacro:property name="supportlen" value="0.07" />
   <xacro:property name="pi" value="3.1415" />
+  <xacro:property name="arm_support_height" value="0.07" />
+  <xacro:property name="arm_support_width" value="0.07" />
+  <xacro:property name="base_arm_len" value="0.2" />
+  <xacro:property name="base_arm_width" value="0.02" />
   <material name="blue">
     <color rgba="0 0 0.8 1"/>
@@ -19,49 +22,46 @@
     </inertial>
   </xacro:macro>
-<!--
-  <xacro:macro name="support" params="prefix reflect">
-    <link name="${prefix}_support">
-      <visual>
-        <geometry>
-          <box size="${supportlen} 0.1 0.2"/>
-        </geometry>
-        <origin xyz="0 0 -${supportlen/2}" rpy="0 ${pi/2} 0"/>
-        <material name="white"/>
-      </visual>
-      <collision>
-        <geometry>
-          <box size="${supportlen} 0.1 0.2"/>
-        </geometry>
-        <origin xyz="0 0 -${supportlen/2}" rpy="0 ${pi/2} 0"/>
-      </collision>
-      <xacro:default_inertial mass="10"/>
-    </link>
-    <joint name="base_to_${prefix}_support" type="fixed">
-      <parent link="main_base"/>
-      <child link="${prefix}_support"/>
-      <origin xyz="0 ${reflect*(main_base_width+.02)} 0.25" />
-    </joint>
-    <link name="${prefix}_base">
-      <visual>
-        <geometry>
-          <box size="${main_base_dims} 0.1 0.1"/>
-        </geometry>
-        <material name="white"/>
-      </visual>
-      <collision>
-        <geometry>
-          <box size="${main_base_dims} 0.1 0.1"/>
-        </geometry>
-      </collision>
-      <xacro:default_inertial mass="10"/>
-    </link>
-    <joint name="${prefix}_base_joint" type="fixed">
-      <parent link="${prefix}_support"/>
-      <child link="${prefix}_base"/>
-      <origin xyz="0 0 ${-supportlen}" />
-    </joint>
-  </xacro:macro>
-  <xacro:support prefix="right" reflect="-1" />
-  <xacro:support prefix="left" reflect="1" /> -->
+  <link name="base_arm">
+    <visual>
+      <geometry>
+        <cylinder radius="${base_arm_width}" length="${base_arm_len}"/>
+      </geometry>
+      <material name="blue"/>
+      <origin xyz="${base_arm_width} 0 ${ base_arm_len/2}"/>
+    </visual>
+    <collision>
+      <geometry>
+        <cylinder radius="${main_base_width}" length="${main_base_bodylen}"/>
+      </geometry>
+    </collision>
+    <xacro:default_inertial mass="10"/>
+  </link>
+  <joint name="base_arm_to_base_arm_support" type="continuous">
+    <axis xyz="1 0 0" rpy="0 0 0" />
+    <parent link="base_arm_support"/>
+    <child link="base_arm"/>
+    <origin xyz="0 0 ${(main_base_bodylen + main_base_height )}"/>
+  </joint>
+  <link name="base_arm_support">
+    <visual>
+      <geometry>
+        <box size="0.01 0.1 ${arm_support_height}"/>
+      </geometry>
+      <material name="blue"/>
+      <origin xyz="0 0 ${(main_base_bodylen ) + main_base_height }"/>
+    </visual>
+    <collision>
+      <geometry>
+        <box size="${main_base_dims} ${main_base_dims} ${main_base_dims}"/>
+      </geometry>
+    </collision>
+    <xacro:default_inertial mass="10"/>
+  </link>
+  <joint name="base_arm_support_to_main_base" type="fixed">
+    <axis xyz="0 0 1" rpy="0 0 0" />
+    <parent link="main_base"/>
+    <child link="base_arm_support"/>
+    <origin xyz="0 0 0"/>
+  </joint>
   <link name="main_base">
     <visual>
@@ -70,5 +70,5 @@
       </geometry>
       <material name="blue"/>
-      <origin xyz="0 0 ${(main_base_bodylen/2.0) + main_base_height }"/>
+      <origin xyz="0 0 ${(main_base_bodylen/2.0) + (main_base_height/2.0) }"/>
     </visual>
     <collision>

Commit message: added eblow and rename

File: urdf/sainsmart_6dof.urdf.xacro (robot description, xacro)
@@ -22,4 +22,25 @@
     </inertial>
   </xacro:macro>
+  <link name="elbow">
+    <visual>
+      <geometry>
+        <box size="0.05 0.05 ${arm_support_height}"/>
+      </geometry>
+      <material name="blue"/>
+      <origin xyz="0 0 0"/>
+    </visual>
+    <collision>
+      <geometry>
+        <box size="${main_base_dims} ${main_base_dims} ${main_base_dims}"/>
+      </geometry>
+    </collision>
+    <xacro:default_inertial mass="10"/>
+  </link>
+  <joint name="eblow" type="continuous">
+    <axis xyz="1 0 0" rpy="0 0 0" />
+    <parent link="base_arm"/>
+    <child link="elbow"/>
+    <origin xyz="0 0 ${ base_arm_len }"/>
+  </joint>
   <link name="base_arm">
     <visual>
@@ -37,5 +58,5 @@
     <xacro:default_inertial mass="10"/>
   </link>
-  <joint name="base_arm_to_base_arm_support" type="continuous">
+  <joint name="shoulder" type="continuous">
     <axis xyz="1 0 0" rpy="0 0 0" />
     <parent link="base_arm_support"/>
@@ -94,5 +115,5 @@
     <xacro:default_inertial mass="10"/>
   </link>
-  <joint name="base_link_to_main_base" type="continuous">
+  <joint name="base" type="continuous">
     <axis xyz="0 0 1" rpy="0 0 0" />
     <parent link="base_link"/>

Commit message: adding wrist... little funky

File: urdf/sainsmart_6dof.urdf.xacro (robot description, xacro)
@@ -1,13 +1,20 @@
 <?xml version="1.0"?>
 <robot name="sainsmart" xmlns:xacro="http://ros.org/wiki/xacro">
+  <!-- constants -->
+  <xacro:property name="pi" value="3.1415" />
+<!-- arm properties -->
   <xacro:property name="main_base_width" value="0.05" />
   <xacro:property name="main_base_bodylen" value="0.06" />
   <xacro:property name="main_base_dims" value="0.1" />
   <xacro:property name="main_base_height" value="0.01" />
-  <xacro:property name="pi" value="3.1415" />
   <xacro:property name="arm_support_height" value="0.07" />
   <xacro:property name="arm_support_width" value="0.07" />
   <xacro:property name="base_arm_len" value="0.2" />
   <xacro:property name="base_arm_width" value="0.02" />
+  <xacro:property name="forearm_len" value="0.15" />
+  <xacro:property name="forearm_width" value="0.02" />
+  <xacro:property name="wrist_len" value="0.15" />
+  <xacro:property name="wrist_width" value="0.02" />
+  <!-- Materials -->
   <material name="blue">
     <color rgba="0 0 0.8 1"/>
@@ -16,4 +23,5 @@
     <color rgba="1 1 1 1"/>
   </material>
+  <!-- Macros -->
   <xacro:macro name="default_inertial" params="mass">
     <inertial>
@@ -22,4 +30,46 @@
     </inertial>
   </xacro:macro>
+  <link name="wrist">
+    <visual>
+      <geometry>
+        <cylinder radius="${wrist_width }" length="${wrist_len}"/>
+      </geometry>
+      <material name="blue"/>
+      <origin xyz=" 0 ${forearm_len/2} 0" rpy="${pi/2}  0 0 "/>
+    </visual>
+    <collision>
+      <geometry>
+        <cylinder radius="${wrist_width}" length="${wrist_len}"/>
+      </geometry>
+    </collision>
+    <xacro:default_inertial mass="10"/>
+  </link>
+  <joint name="wrist" type="continuous">
+    <axis xyz=" 0 1  0" rpy="0 0 0" />
+    <parent link="forearm"/>
+    <child link="wrist"/>
+    <origin xyz="0 ${wrist_len} 0"/>
+  </joint>
+  <link name="forearm">
+    <visual>
+      <geometry>
+        <cylinder radius="${forearm_width }" length="${forearm_len}"/>
+      </geometry>
+      <material name="blue"/>
+      <origin xyz=" 0 ${forearm_len/2} 0" rpy="${pi/2}  0 0 "/>
+    </visual>
+    <collision>
+      <geometry>
+        <cylinder radius="${forearm_width }" length="${forearm_len}"/>
+      </geometry>
+    </collision>
+    <xacro:default_inertial mass="10"/>
+  </link>
+  <joint name="roll" type="continuous">
+    <axis xyz=" 0 1  0" rpy="0 0 0" />
+    <parent link="elbow"/>
+    <child link="forearm"/>
+    <origin xyz="0 0 0"/>
+  </joint>
   <link name="elbow">
     <visual>

Commit message: added wrist

File: urdf/sainsmart_6dof.urdf.xacro (robot description, xacro)
@@ -14,5 +14,5 @@
   <xacro:property name="forearm_len" value="0.15" />
   <xacro:property name="forearm_width" value="0.02" />
-  <xacro:property name="wrist_len" value="0.15" />
+  <xacro:property name="wrist_len" value="0.03" />
   <xacro:property name="wrist_width" value="0.02" />
   <!-- Materials -->
@@ -30,4 +30,5 @@
     </inertial>
   </xacro:macro>
+<!-- Wrist -->
   <link name="wrist">
     <visual>
@@ -36,5 +37,5 @@
       </geometry>
       <material name="blue"/>
-      <origin xyz=" 0 ${forearm_len/2} 0" rpy="${pi/2}  0 0 "/>
+      <origin xyz=" 0 0 0" rpy="  0 ${pi/2} 0 "/>
     </visual>
     <collision>
@@ -46,9 +47,10 @@
   </link>
   <joint name="wrist" type="continuous">
-    <axis xyz=" 0 1  0" rpy="0 0 0" />
+    <axis xyz="1 0 0" rpy="0  ${pi/4} 0" />
     <parent link="forearm"/>
     <child link="wrist"/>
-    <origin xyz="0 ${wrist_len} 0"/>
+    <origin xyz="0  ${forearm_len}  0"/>
   </joint>
+<!-- Forearm -->
   <link name="forearm">
     <visual>
@@ -129,5 +131,5 @@
     <xacro:default_inertial mass="10"/>
   </link>
-  <joint name="base_arm_support_to_main_base" type="fixed">
+  <joint name="support" type="fixed">
     <axis xyz="0 0 1" rpy="0 0 0" />
     <parent link="main_base"/>
@@ -165,5 +167,5 @@
     <xacro:default_inertial mass="10"/>
   </link>
-  <joint name="base" type="continuous">
+  <joint name="bottom" type="continuous">
     <axis xyz="0 0 1" rpy="0 0 0" />
     <parent link="base_link"/>

Commit message: finished interface

File: urdf/sainsmart_6dof.urdf.xacro (robot description, xacro)
@@ -16,4 +16,6 @@
   <xacro:property name="wrist_len" value="0.03" />
   <xacro:property name="wrist_width" value="0.02" />
+  <xacro:property name="interface_len" value="0.03" />
+  <xacro:property name="interface_width" value="0.02" />
   <!-- Materials -->
   <material name="blue">
@@ -31,4 +33,27 @@
   </xacro:macro>
 <!-- Wrist -->
+  <link name="interface">
+    <visual>
+      <geometry>
+        <cylinder radius="${interface_width }" length="${interface_len}"/>
+      </geometry>
+      <material name="blue"/>
+      <origin xyz=" 0 0 0" rpy=" ${pi/2} 0     0 "/>
+    </visual>
+    <collision>
+      <geometry>
+        <cylinder radius="${interface_width}" length="${interface_len}"/>
+      </geometry>
+    </collision>
+    <xacro:default_inertial mass="10"/>
+  </link>
+  <joint name="interface" type="revolute">
+    <axis xyz="0 1 0" rpy="${pi/2} 0   0" />
+    <limit effort="0.0001" velocity="0.0001" lower="-2.2" upper="1.7"/>
+    <parent link="wrist"/>
+    <child link="interface"/>
+    <origin xyz="0  ${wrist_width}  0"/>
+  </joint>
+<!-- Wrist -->
   <link name="wrist">
     <visual>
